File: kicad/copv2.kicad_pcb (KiCad board)
At the start: 2 copper layers, 30 x 42 mm, 33 parts, among them J1 Conn_02x03_Counter_Clockwise, Q1 DMP3098LSD-13, U1 ATtiny84A-SS, U2 LM393, U3 LM78M05_TO252

Commit message: mosfet wrong way around
Parts:
- turned Q1 to -90 degrees
- turned R8 to 0 degrees
- renumbered GND to GND1, VCC to VCC1
Connections:
- Q1 pad 1: /IGN1 -> +5V
- Q1 pad 3: /IGN2 -> +5V
- Q1 pad 5: +5V -> /IGN1
- Q1 pad 6: +5V -> /IGN1
- Q1 pad 7: +5V -> /IGN2
- Q1 pad 8: +5V -> /IGN2
Routing:
- net Net-(Q1B-G2): track 10.4 -> 13.3 mm
- net /IGN1: track 14.4 -> 16.7 mm
- net Net-(Q1A-G1): track 11.3 -> 13.3 mm
- net Net-(U1-PA1): track 4.65 -> 3.05 mm
- net /IGN2: track 18.2 -> 19.5 mm
- net +5V: track 59.4 -> 58.9 mm, vias 4 -> 3
