File: kicad/v3/coilonplugv3.kicad_sch (KiCad schematic)
At the start: 32 parts, among them J1 Conn_02x03_Counter_Clockwise, Q1 DMP3098LSD-13, U1 ATtiny84A-SS, U2 SN74LVC1G17DBVR, U3 SN74LVC1G17DBVR, U4 L78L05_SOT89

Commit message: small pcb changes + get code from latest pcb made
Parts:
- R1, R2, R3, R4: LCSC Part # C98220 -> C116677
- U4: LCSC Part # (none) -> C42738
Changed lines of the file:
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@@
 			)
 		)
-		(property "LCSC Part #" "C98220"
+		(property "LCSC Part #" "C116677"
 			(at 119.38 127 90)
 			(hide yes)
@@
 			)
 		)
-		(property "LCSC Part #" "C98220"
+		(property "LCSC Part #" "C116677"
 			(at 119.38 102.87 90)
 			(hide yes)
@@
 			)
 		)
-		(property "LCSC Part #" "C98220"
+		(property "LCSC Part #" "C116677"
 			(at 45.72 40.64 90)
 			(hide yes)
@@
 			)
 		)
+		(property "LCSC Part #" "C42738"
+			(at 162.56 76.2 0)
+			(hide yes)
+			(show_name no)
+			(do_not_autoplace no)
+			(effects
+				(font
+					(size 1.27 1.27)
+				)
+			)
+		)
 		(pin "1"
 		)
@@
 			)
 		)
-		(property "LCSC Part #" "C98220"
+		(property "LCSC Part #" "C116677"
 			(at 45.72 74.93 90)
 			(hide yes)

Commit message: capacitor brand change before order
Parts:
- C2: LCSC Part # C107070 -> C354382
Changed lines of the file:
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@@
 			)
 		)
-		(property "LCSC Part #" "C107070"
+		(property "LCSC Part #" "C354382"
 			(at 146.05 80.01 0)
 			(hide yes)
