File: kicad/v3/coilonplugv3.kicad_pcb (KiCad board)
At the start: 2 copper layers, 26.2 x 33.4 mm, 32 parts, among them J1 Conn_02x03_Counter_Clockwise, Q1 DMP3098LSD-13, U1 ATtiny84A-SS, U2 SN74LVC1G17DBVR, U3 SN74LVC1G17DBVR, U4 L78L05_SOT89

Commit message: small pcb changes + get code from latest pcb made
Routing:
- net GND: vias 29 -> 32
Changed lines of the file:
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@@
 	)
 	(setup
+		(stackup
+			(layer "F.SilkS"
+				(type "Top Silk Screen")
+				(color "White")
+			)
+			(layer "F.Paste"
+				(type "Top Solder Paste")
+			)
+			(layer "F.Mask"
+				(type "Top Solder Mask")
+				(color "Black")
+				(thickness 0.01)
+			)
+			(layer "F.Cu"
+				(type "copper")
+				(thickness 0.035)
+			)
+			(layer "dielectric 1"
+				(type "core")
+				(thickness 1.51)
+				(material "FR4")
+				(epsilon_r 4.5)
+				(loss_tangent 0.02)
+			)
+			(layer "B.Cu"
+				(type "copper")
+				(thickness 0.035)
+			)
+			(layer "B.Mask"
+				(type "Bottom Solder Mask")
+				(color "Black")
+				(thickness 0.01)
+			)
+			(layer "B.Paste"
+				(type "Bottom Solder Paste")
+			)
+			(layer "B.SilkS"
+				(type "Bottom Silk Screen")
+				(color "White")
+			)
+			(copper_finish "None")
+			(dielectric_constraints no)
+		)
 		(pad_to_mask_clearance 0)
 		(allow_soldermask_bridges_in_footprints no)
@@
 			)
 		)
-		(property "LCSC Part #" "C98220"
+		(property "LCSC Part #" "C116677"
 			(at 0 0 180)
 			(unlocked yes)
@@
 			)
 		)
-		(property "LCSC Part #" "C98220"
+		(property "LCSC Part #" "C116677"
 			(at 0 0 180)
 			(unlocked yes)
@@
 		(tags "SOT-89-3")
 		(property "Reference" "U4"
-			(at 3.6375 -3.25 0)
+			(at 3.2375 -2.85 0)
 			(layer "F.SilkS")
 			(effects
@@
 			)
 		)
+		(property "LCSC Part #" "C42738"
+			(at 0 0 180)
+			(unlocked yes)
+			(layer "F.Fab")
+			(hide yes)
+			(effects
+				(font
+					(size 1 1)
+					(thickness 0.15)
+				)
+			)
+		)
 		(property ki_fp_filters "SOT?89*")
 		(sheetname "/")
@@
 			)
 		)
-		(property "LCSC Part #" "C98220"
+		(property "LCSC Part #" "C116677"
 			(at 0 0 270)
 			(unlocked yes)
@@
 		(tags "capacitor")
 		(property "Reference" "C1"
-			(at 2.5 0 180)
+			(at 2.15 0.05 180)
 			(layer "F.SilkS")
 			(effects
@@
 			)
 		)
-		(property "LCSC Part #" "C98220"
+		(property "LCSC Part #" "C116677"
 			(at 0 0 90)
 			(unlocked yes)
@@
 	)
 	(via
+		(at 178 74.75)
+		(size 0.6)
+		(drill 0.3)
+		(layers "F.Cu" "B.Cu")
+		(free yes)
+		(net "GND")
+	)
+	(via
 		(at 183 105.25)
 		(size 0.6)
@@
 	)
 	(via
+		(at 179.75 74.8)
+		(size 0.6)
+		(drill 0.3)
+		(layers "F.Cu" "B.Cu")
+		(free yes)
+		(net "GND")
+	)
+	(via
 		(at 178 104.9)
 		(size 0.6)
@@
 		(net "GND")
 	)
+	(via
+		(at 178.9 76.5)
+		(size 0.6)
+		(drill 0.3)
+		(layers "F.Cu" "B.Cu")
+		(net "GND")
+	)

Commit message: test failed, try new code
Routing:
- net GND: vias 32 -> 30
Changed lines of the file:
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@@
 	)
 	(via
-		(at 180.5 106)
+		(at 179.7 105.2)
 		(size 0.6)
 		(drill 0.3)
@@
 	)
 	(via
-		(at 180.4 103.6)
+		(at 180.05 103.3)
 		(size 0.6)
 		(drill 0.3)
@@
 	(via
 		(at 178.3 99)
-		(size 0.6)
-		(drill 0.3)
-		(layers "F.Cu" "B.Cu")
-		(free yes)
-		(net "GND")
-	)
-	(via
-		(at 173.15 104.55)
 		(size 0.6)
 		(drill 0.3)
@@
 		(size 0.6)
 		(drill 0.3)
-		(layers "F.Cu" "B.Cu")
-		(free yes)
-		(net "GND")
-	)
-	(via
-		(at 178 104.9)
-		(size 0.6)
-		(drill 0.3)

Commit message: ordered! state of repository when pcb ordered
Routing:
- net /IGN2/3Filtered: track 15.6 -> 17.1 mm
Changed lines of the file:
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@@
-	)
-	(segment
-		(start 174.8 78.524999)
-		(end 174.8 82.55)
-		(width 0.2)
-		(layer "F.Cu")
-		(net "/IGN2{slash}3Filtered")
 	)
 	(segment
@@
 	)
 	(segment
-		(start 172.5 75.25)
-		(end 172.5 76.224999)
-		(width 0.2)
-		(layer "F.Cu")
-		(net "/IGN2{slash}3Filtered")
-	)
-	(segment
 		(start 171.5625 86.95)
 		(end 172.0625 87.45)
@@
 	)
 	(segment
-		(start 172.5 76.224999)
-		(end 174.8 78.524999)
+		(start 172.5 75.975)
+		(end 172.5 75.25)
+		(width 0.2)
+		(layer "F.Cu")
+		(net "/IGN2{slash}3Filtered")
+	)
+	(segment
+		(start 171.875 81.4)
+		(end 171.875 76.6)
+		(width 0.2)
+		(layer "F.Cu")
+		(net "/IGN2{slash}3Filtered")
+	)
+	(segment
+		(start 172.25 81.775)
+		(end 171.875 81.4)
+		(width 0.2)
+		(layer "F.Cu")
+		(net "/IGN2{slash}3Filtered")
+	)
+	(segment
+		(start 174.8 82.55)
+		(end 174.025 81.775)
+		(width 0.2)
+		(layer "F.Cu")
+		(net "/IGN2{slash}3Filtered")
+	)
+	(segment
+		(start 174.025 81.775)
+		(end 172.25 81.775)
+		(width 0.2)
+		(layer "F.Cu")
+		(net "/IGN2{slash}3Filtered")
+	)
+	(segment
+		(start 171.875 76.6)
+		(end 172.5 75.975)
 		(width 0.2)
 		(layer "F.Cu")
@@
 	)
 	(segment
+		(start 180.5 96.2)
+		(end 184.1 92.6)
+		(width 0.5)
+		(layer "B.Cu")
+		(net "VCC")
+	)
+	(segment
 		(start 184.1 75.6)
 		(end 183.3 74.8)
@@
 	)
 	(segment
-		(start 180.5 96.2)
-		(end 184.1 92.6)
-		(width 0.5)
-		(layer "B.Cu")
-		(net "VCC")
-	)
-	(segment
 		(start 161.3 84.6)
 		(end 161.3 84.7)
@@
 	)
 	(segment
-		(start 171.23 76.044448)
-		(end 168.02 79.254448)
-		(width 0.2)
-		(layer "F.Cu")
-		(net "/IGN1{slash}4Filtered")
-	)
-	(segment
-		(start 166.635552 82.6)
-		(end 166.05 82.6)
-		(width 0.2)
-		(layer "F.Cu")
-		(net "/IGN1{slash}4Filtered")
-	)
-	(segment
 		(start 171.23 75.25)
 		(end 171.23 76.044448)
@@
 	)
 	(segment
-		(start 168.02 79.254448)
-		(end 168.02 81.215552)
+		(start 166.7 82.6)
+		(end 166.05 82.6)
+		(width 0.2)
+		(layer "F.Cu")
+		(net "/IGN1{slash}4Filtered")
+	)
+	(segment
+		(start 168.05 81.25)
+		(end 166.7 82.6)
+		(width 0.2)
+		(layer "F.Cu")
+		(net "/IGN1{slash}4Filtered")
+	)
+	(segment
+		(start 168.05 79.224448)
+		(end 168.05 81.25)
+		(width 0.2)
+		(layer "F.Cu")
+		(net "/IGN1{slash}4Filtered")
+	)
+	(segment
+		(start 171.23 76.044448)
+		(end 168.05 79.224448)
 		(width 0.2)
 		(layer "F.Cu")
@@
 		(net "/IGN1{slash}4Filtered")
 	)
-	(segment
-		(start 168.02 81.215552)
-		(end 166.635552 82.6)
-		(width 0.2)
-		(layer "F.Cu")
-		(net "/IGN1{slash}4Filtered")
-	)
 	(via
 		(at 166.05 82.6)
@@
 	)
 	(segment
+		(start 173.4 88.3)
+		(end 175.88 88.3)
+		(width 0.2)
+		(layer "F.Cu")
+		(net "Net-(Q1B-G2)")
+	)
+	(segment
 		(start 182.8 85.375)
 		(end 183.75 86.325)
@@
 	)
 	(segment
+		(start 169.325 79.025)
+		(end 169.325 82.575)
+		(width 0.2)
+		(layer "F.Cu")
+		(net "Net-(Q1B-G2)")
+	)
+	(segment
+		(start 169.65 78.7)
+		(end 169.325 79.025)
+		(width 0.2)
+		(layer "F.Cu")
+		(net "Net-(Q1B-G2)")
+	)
+	(segment
+		(start 178.75 83.95)
+		(end 179.9 82.8)
+		(width 0.2)
+		(layer "F.Cu")
+		(net "Net-(Q1B-G2)")
+	)
+	(segment
+		(start 171.45 84.7)
+		(end 172.8 84.7)
+		(width 0.2)
+		(layer "F.Cu")
+		(net "Net-(Q1B-G2)")
+	)
+	(segment
 		(start 173.2 85.1)
 		(end 173.2 88.1)
@@
 	)
 	(segment
+		(start 171.23 79.225001)
+		(end 170.704999 78.7)
+		(width 0.2)
+		(layer "F.Cu")
+		(net "Net-(Q1B-G2)")
+	)
+	(segment
+		(start 175.88 88.3)
+		(end 176.525 87.655)
+		(width 0.2)
+		(layer "F.Cu")
+		(net "Net-(Q1B-G2)")
+	)
+	(segment
+		(start 178.55 87.7)
+		(end 178.75 87.5)
+		(width 0.2)
+		(layer "F.Cu")
+		(net "Net-(Q1B-G2)")
+	)
+	(segment
+		(start 170.704999 78.7)
+		(end 169.65 78.7)
+		(width 0.2)
+		(layer "F.Cu")
+		(net "Net-(Q1B-G2)")
+	)
+	(segment
+		(start 169.325 82.575)
+		(end 171.45 84.7)
+		(width 0.2)
+		(layer "F.Cu")
+		(net "Net-(Q1B-G2)")
+	)
+	(segment
+		(start 182.8 83.3)
+		(end 182.8 85.375)
+		(width 0.2)
+		(layer "F.Cu")
+		(net "Net-(Q1B-G2)")
+	)
+	(segment
+		(start 182.3 82.8)
+		(end 182.8 83.3)
+		(width 0.2)
+		(layer "F.Cu")
+		(net "Net-(Q1B-G2)")
+	)
+	(segment
+		(start 172.8 84.7)
+		(end 173.2 85.1)
+		(width 0.2)
+		(layer "F.Cu")
+		(net "Net-(Q1B-G2)")
+	)
+	(segment
+		(start 179.9 82.8)
+		(end 182.3 82.8)
+		(width 0.2)
+		(layer "F.Cu")
+		(net "Net-(Q1B-G2)")
+	)
+	(segment
+		(start 173.2 88.1)
+		(end 173.4 88.3)
+		(width 0.2)
+		(layer "F.Cu")
+		(net "Net-(Q1B-G2)")
+	)
+	(segment
 		(start 171.23 80.2)
 		(end 171.23 79.225001)
@@
 	)
 	(segment
-		(start 178.75 83.95)
-		(end 179.9 82.8)
-		(width 0.2)
-		(layer "F.Cu")
-		(net "Net-(Q1B-G2)")
-	)
-	(segment
-		(start 175.88 88.3)
-		(end 176.525 87.655)
-		(width 0.2)
-		(layer "F.Cu")
-		(net "Net-(Q1B-G2)")
-	)
-	(segment
-		(start 170.704999 78.7)
-		(end 169.65 78.7)
-		(width 0.2)
-		(layer "F.Cu")
-		(net "Net-(Q1B-G2)")
-	)
-	(segment
-		(start 178.55 87.7)
-		(end 178.75 87.5)
-		(width 0.2)
-		(layer "F.Cu")
-		(net "Net-(Q1B-G2)")
-	)
-	(segment
-		(start 182.8 83.3)
-		(end 182.8 85.375)
-		(width 0.2)
-		(layer "F.Cu")
-		(net "Net-(Q1B-G2)")
-	)
-	(segment
-		(start 173.2 88.1)
-		(end 173.4 88.3)
-		(width 0.2)
-		(layer "F.Cu")
-		(net "Net-(Q1B-G2)")
-	)
-	(segment
-		(start 182.3 82.8)
-		(end 182.8 83.3)
-		(width 0.2)
-		(layer "F.Cu")
-		(net "Net-(Q1B-G2)")
-	)
-	(segment
-		(start 179.9 82.8)
-		(end 182.3 82.8)
-		(width 0.2)
-		(layer "F.Cu")
-		(net "Net-(Q1B-G2)")
-	)
-	(segment
-		(start 173.4 88.3)
-		(end 175.88 88.3)
-		(width 0.2)
-		(layer "F.Cu")
-		(net "Net-(Q1B-G2)")
-	)
-	(segment
-		(start 169.65 78.7)
-		(end 169.35 79)
-		(width 0.2)
-		(layer "F.Cu")
-		(net "Net-(Q1B-G2)")
-	)
-	(segment
 		(start 176.57 87.7)
 		(end 178.55 87.7)
@@
 	)
 	(segment
-		(start 171.23 79.225001)
-		(end 170.704999 78.7)
-		(width 0.2)
-		(layer "F.Cu")
-		(net "Net-(Q1B-G2)")
-	)
-	(segment
-		(start 172.8 84.7)
-		(end 173.2 85.1)
-		(width 0.2)
-		(layer "F.Cu")
-		(net "Net-(Q1B-G2)")
-	)
-	(segment
 		(start 178.75 87.5)
 		(end 178.75 83.95)
@@
 	)
 	(segment
-		(start 169.35 82.6)
-		(end 171.45 84.7)
-		(width 0.2)
-		(layer "F.Cu")
-		(net "Net-(Q1B-G2)")
-	)
-	(segment
-		(start 169.35 79)
-		(end 169.35 82.6)
-		(width 0.2)
-		(layer "F.Cu")
-		(net "Net-(Q1B-G2)")
-	)
-	(segment
-		(start 171.45 84.7)
-		(end 172.8 84.7)
-		(width 0.2)
-		(layer "F.Cu")
-		(net "Net-(Q1B-G2)")
-	)
-	(segment
 		(start 181.475 90.225)
 		(end 183 91.75)
@@
 	)
 	(segment
+		(start 164.1 76.6)
+		(end 169.584999 76.6)
+		(width 0.2)
+		(layer "F.Cu")
+		(net "/RESET")
+	)
+	(segment
 		(start 163.25 75.75)
-		(end 164.025 76.525)
+		(end 164.1 76.6)
 		(width 0.2)
 		(layer "F.Cu")
@@
 	)
 	(segment
-		(start 169.659999 76.525)
+		(start 169.584999 76.6)
 		(end 169.96 76.224999)
 		(width 0.2)
@@
 		(width 0.2)
 		(layer "F.Cu")
-		(net "/RESET")
-	)
-	(segment
-		(start 164.025 76.525)
-		(end 169.659999 76.525)
-		(width 0.2)
-		(layer "F.Cu")
